Commit message: Controller on dev...

File: install/magnetic_robot/share/magnetic_robot/urdf/Magnetic_robot.urdf (robot description, URDF)
Before this commit: robot Robot Arm Assem Materials, 7 links, 6 joints
Links:
- removed link link_3
- removed link link_4
- removed link link_5
- removed link link_6
- link base_link: mass 0.198830632182665 -> 1.8830632182665; geometry collision mesh filename=package://magnetic_robot/meshes/base_link.STL; visual mesh filename=package://magnetic_robot/meshes/base_link.STL
- link link_1: geometry collision mesh filename=package://magnetic_robot/meshes/link_1.STL; visual mesh filename=package://magnetic_robot/meshes/link_1.STL
- link link_2: mass 0.029523127189033 -> 0.059523127189033; geometry collision mesh filename=package://magnetic_robot/meshes/link_2.STL; visual mesh filename=package://magnetic_robot/meshes/link_2.STL
Joints:
- removed joint joint_23
- removed joint joint_34
- removed joint joint_45
- removed joint joint_56
- joint joint_12: origin xyz=0.009 -0.0075 0.025 rpy=0 1.5708 0 -> xyz=0.009 -0.0075 0.025 rpy=0 1.5707963267949 0

File: src/magnetic_robot/urdf/Magnetic_robot.urdf (robot description, URDF)
Before this commit: robot magnetic_robot, 7 links, 6 joints
Links:
- removed link link_3
- removed link link_4
- removed link link_5
- removed link link_6
Joints:
- removed joint joint_23
- removed joint joint_34
- removed joint joint_45
- removed joint joint_56
