Commit message: Added simulink model

File: install/magnetic_robot/share/magnetic_robot/urdf/Magnetic_robot_effort.urdf (robot description, URDF)
Before this commit: robot magnetic_robot, 8 links, 7 joints
Links:
- link base_link: mass 1.8830632182665 -> 0.198830632182665

Commit message: Fixed Simulink model

File: install/magnetic_robot/share/magnetic_robot/urdf/Magnetic_robot_effort.urdf (robot description, URDF)
Before this commit: robot magnetic_robot, 8 links, 7 joints
Joints:
- joint joint_12: limit lower=-3.1416 upper=3.1416 effort=1000 velocity=19 -> lower=0 upper=0 effort=1000 velocity=19
- joint joint_23: limit lower=-3.1416 upper=3.1416 effort=1000 velocity=10 -> lower=0 upper=0 effort=1000 velocity=10
- joint joint_34: limit lower=-3.1416 upper=3.1416 effort=1000 velocity=10 -> lower=0 upper=0 effort=1000 velocity=10
- joint joint_45: limit lower=-3.1416 upper=3.1416 effort=1000 velocity=10 -> lower=0 upper=0 effort=1000 velocity=10
